Commit message: add dependencies bash files

File: robots/LoCoBot/locobot_description/urdf/d435.urdf.xacro (robot description, xacro)
@@ -46,5 +46,5 @@
         <geometry>
           <!-- <box size="${d435_cam_width} ${d435_cam_height} ${d435_cam_depth}"/> -->
-	  <mesh filename="package://realsense2_camera/meshes/d435.dae" />
+	  <mesh filename="package://locobot_description/meshes/d435.dae" />
           <!--<mesh filename="package://realsense2_camera/meshes/d435/d435.dae" />-->
         </geometry>
